File: hamusb.kicad_pcb (KiCad board)
At the start: 2 copper layers, 37.5 x 17.5 mm, 20 parts, among them P1 USB, P2 DATA, Q1 2N7002E, U1 FT232RL, U2 74AC125, Y1 12MHz

Commit message: Replaced USB receptable with USB plug
Parts:
- P1: footprint Connect:USB_A -> USB_A_M
- moved JP3 11.0 mm to (131.8, 99.0), turned to 90 degrees
- moved P1 4.43 mm to (128.6, 105.8)
- turned L1 to 180 degrees
Connections:
- L1 pad 1: Net-(C4-Pad1) -> VCC
- L1 pad 2: VCC -> Net-(C4-Pad1)
Routing:
- net Earth: track 43.1 -> 4.20 mm
- net Net-(C4-Pad1): track 15.0 -> 23.5 mm
- net Net-(P1-Pad2): track 13.0 -> 14.2 mm
- net GND: track 23.3 -> 24.0 mm
- added copper zone on B.Cu, net Earth
