File: hamusb.sch (KiCad schematic (older format))
At the start: 20 parts, among them P1 USB, P2 DATA, Q1 2N7002E, U1 FT232RL, U2 74AC125, Y1 12MHz

Commit message: Replaced USB receptable with USB plug
Parts:
- P1: footprint Connect:USB_A -> onitake:USB_A_M
Changed lines of the file:
@@
 F 0 "P1" H 3600 2950 50  0000 C CNN
 F 1 "USB" H 3350 3350 50  0000 C CNN
-F 2 "Connect:USB_A" V 3350 3050 60  0001 C CNN
+F 2 "onitake:USB_A_M" V 3350 3050 60  0001 C CNN
 F 3 "" V 3350 3050 60  0000 C CNN
 	1    3400 3150
